Commit message: Arm story, checkpoint 5: two cells side by side in one world
Side by side is built as ONE Gazebo world with two UR5e cells, not two
synchronised simulators. One physics clock means the runs are frame
locked by construction; two simulators would drift and the comparison
would be worthless. It is also half the GPU and records as one window.

  models      ground_plane, panel_left, panel_right, ur5e_left, ur5e_right
  left cell   arm_controller + joint_state_broadcaster active
  right cell  arm_controller + joint_state_broadcaster active
  cameras     /left/camera/image and /right/camera/image, 6 blobs each

The robot xacro is now parameterised by prefix and namespace, with a
controllers yaml per side.

One more failure worth recording: prefixing the base link to left_world
broke it. A link named exactly "world" is the URDF convention that
anchors a robot to the global frame; renaming it made the arm a free
floating body that drifted off its spawn point, measured at
(0, 0.172, 0.206) instead of the origin, which put both panels out of
frame. Link names are model scoped in Gazebo, so both robots can keep a
link called "world".

Known caveat: with the base link unprefixed, both robot_state_publishers
publish from a frame called "world" while Gazebo places the models at
different x. TF for the right cell is therefore offset. The guard and the
control loop work in image coordinates and do not use TF, so this does
not affect the demo, but it would need fixing before anyone trusted TF
here.

File: ros2_ws/src/blindspot_arm/urdf/ur5e_camera.urdf.xacro (robot description, xacro)
@@ -8,9 +8,18 @@
   <xacro:arg name="ur_type" default="ur5e"/>
   <xacro:arg name="name" default="ur"/>
+  <xacro:arg name="prefix" default=""/>
+  <xacro:arg name="ns" default=""/>
+  <xacro:arg name="controllers_file"
+             default="$(find blindspot_arm)/config/controllers.yaml"/>
+  <!-- must be named exactly "world": that is the URDF convention that
+       anchors the base to the global frame. Prefixing it made the arm a
+       free-floating body which drifted off its spawn point (measured
+       ur5e_left at 0,0.172,0.206 instead of the origin). Link names are
+       model-scoped in Gazebo, so both robots can have one. -->
   <link name="world"/>
   <xacro:include filename="$(find ur_description)/urdf/ur_macro.xacro"/>
   <xacro:ur_robot
       name="$(arg name)"
-      tf_prefix=""
+      tf_prefix="$(arg prefix)"
       parent="world"
       joint_limits_parameters_file="$(find ur_description)/config/$(arg ur_type)/joint_limits.yaml"
@@ -21,5 +30,5 @@
   </xacro:ur_robot>
   <!-- eye in hand: camera rigidly attached to tool0, looking along +z -->
-  <link name="camera_link">
+  <link name="$(arg prefix)camera_link">
     <visual>
       <geometry><box size="0.03 0.06 0.03"/></geometry>
@@ -32,23 +41,23 @@
     </inertial>
   </link>
-  <joint name="camera_joint" type="fixed">
-    <parent link="tool0"/>
-    <child link="camera_link"/>
+  <joint name="$(arg prefix)camera_joint" type="fixed">
+    <parent link="$(arg prefix)tool0"/>
+    <child link="$(arg prefix)camera_link"/>
     <origin xyz="0 0 0.02" rpy="0 0 0"/>
   </joint>
   <!-- optical frame: computer-vision convention, +z forward, +y down.
        The guard works in normalised image coordinates in THIS frame. -->
-  <link name="camera_optical_frame"/>
-  <joint name="camera_optical_joint" type="fixed">
-    <parent link="camera_link"/>
-    <child link="camera_optical_frame"/>
+  <link name="$(arg prefix)camera_optical_frame"/>
+  <joint name="$(arg prefix)camera_optical_joint" type="fixed">
+    <parent link="$(arg prefix)camera_link"/>
+    <child link="$(arg prefix)camera_optical_frame"/>
     <origin xyz="0 0 0" rpy="${-pi/2} 0 ${-pi/2}"/>
   </joint>
-  <ros2_control name="GzSystem" type="system">
+  <ros2_control name="$(arg prefix)GzSystem" type="system">
     <hardware>
       <plugin>gz_ros2_control/GazeboSimSystem</plugin>
     </hardware>
     <xacro:macro name="jnt" params="n init">
-      <joint name="${n}">
+      <joint name="$(arg prefix)${n}">
         <command_interface name="position"/>
         <state_interface name="position"><param name="initial_value">${init}</param></state_interface>
@@ -67,20 +76,21 @@
     <plugin filename="gz_ros2_control-system"
             name="gz_ros2_control::GazeboSimROS2ControlPlugin">
-      <parameters>$(find blindspot_arm)/config/controllers.yaml</parameters>
+      <parameters>$(arg controllers_file)</parameters>
+      <ros><namespace>$(arg ns)</namespace></ros>
     </plugin>
   </gazebo>
-  <gazebo reference="camera_link">
-    <sensor name="wrist_camera" type="camera">
+  <gazebo reference="$(arg prefix)camera_link">
+    <sensor name="$(arg prefix)wrist_camera" type="camera">
       <camera>
         <horizontal_fov>1.0472</horizontal_fov>
         <image><width>640</width><height>480</height><format>R8G8B8</format></image>
         <clip><near>0.02</near><far>10.0</far></clip>
-        <optical_frame_id>camera_optical_frame</optical_frame_id>
+        <optical_frame_id>$(arg prefix)camera_optical_frame</optical_frame_id>
       </camera>
       <always_on>1</always_on>
       <update_rate>20</update_rate>
       <visualize>false</visualize>
-      <topic>wrist_camera</topic>
-      <gz_frame_id>camera_optical_frame</gz_frame_id>
+      <topic>$(arg prefix)wrist_camera</topic>
+      <gz_frame_id>$(arg prefix)camera_optical_frame</gz_frame_id>
     </sensor>
   </gazebo>
